File: hardware/Gigaspark_Mega/Gigaspark_Mega.kicad_sch (KiCad schematic)
At the start: 0 parts

Commit message: KiCad Bloque 2: Frontal Analogico - Osciloscopio + Multimetro + Proteccion
Other:
- title: Gigaspark Mega - Bloque 1: MCU, Storage, Audio, Power -> Gigaspark Mega - Bloque 2: Frontal Analogico (Osciloscopio + Multimetro)
Changed lines of the file:
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@@
   (paper "A3")
   (title_block
-    (title "Gigaspark Mega - Bloque 1: MCU, Storage, Audio, Power")
+    (title "Gigaspark Mega - Bloque 2: Frontal Analogico (Osciloscopio + Multimetro)")
     (date "2026-09-07")
     (rev "1.0")
     (comment 1 "Gigaspark OS - Mega Device")
-    (comment 2 "Bloque 1: Base MCU + IO")
+    (comment 2 "Bloque 2: Analog Frontend - Protection + Signal Conditioning")
   )
-  (junction (at 0 0) (diameter 0) (color 0 0 0 0) (uuid "j0000001-0001-0001-0001-000000000001"))
   (sheet_instances
     (path "/" (page "1"))

Commit message: KiCad Bloque 3: Fuente Dual 30V/5A + Serie/Paralelo + MCP41010
Other:
- title: Gigaspark Mega - Bloque 2: Frontal Analogico (Osciloscopio + Multimetro) -> Gigaspark Mega - Bloque 3: Fuente Dual 30V/5A
Changed lines of the file:
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@@
   (paper "A3")
   (title_block
-    (title "Gigaspark Mega - Bloque 2: Frontal Analogico (Osciloscopio + Multimetro)")
+    (title "Gigaspark Mega - Bloque 3: Fuente Dual 30V/5A")
     (date "2026-09-07")
     (rev "1.0")
     (comment 1 "Gigaspark OS - Mega Device")
-    (comment 2 "Bloque 2: Analog Frontend - Protection + Signal Conditioning")
+    (comment 2 "Bloque 3: Dual Power Supply + Series/Parallel")
   )
   (sheet_instances

Commit message: KiCad Bloque 4: RF Tools (CC1101+PN532+IR) + Controles Fisicos (D-Pad)
Other:
- title: Gigaspark Mega - Bloque 3: Fuente Dual 30V/5A -> Gigaspark Mega - Bloque 4: RF Tools + Physical Controls
Changed lines of the file:
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@@
   (paper "A3")
   (title_block
-    (title "Gigaspark Mega - Bloque 3: Fuente Dual 30V/5A")
+    (title "Gigaspark Mega - Bloque 4: RF Tools + Physical Controls")
     (date "2026-09-07")
     (rev "1.0")
     (comment 1 "Gigaspark OS - Mega Device")
-    (comment 2 "Bloque 3: Dual Power Supply + Series/Parallel")
+    (comment 2 "Bloque 4: CC1101 + PN532 + IR + D-Pad + Buttons")
   )
   (sheet_instances
